Commit message: Remove unneeded urdf tags for hyqreal to be able to work with Pinocchio

File: resources/urdfs/hyqreal/urdf/hyqreal.urdf (robot description, URDF)
Before this commit: robot hyqreal, 43 links, 42 joints
Links:
- link base_link: geometry 
- link lf_foot: geometry 
- link lf_hipassembly: geometry 
- link lf_lowerleg: geometry 
- link lf_upperleg: geometry 
- link lh_foot: geometry 
- link lh_hipassembly: geometry 
- link lh_lowerleg: geometry 
- link lh_upperleg: geometry 
- link realsense/back/camera_link: geometry 
- link realsense/front/camera_link: geometry 
- link rf_foot: geometry 
- link rf_hipassembly: geometry 
- link rf_lowerleg: geometry 
- link rf_upperleg: geometry 
- link rh_foot: geometry 
- link rh_hipassembly: geometry 
- link rh_lowerleg: geometry 
- link rh_upperleg: geometry 
- link trunk: geometry 
- link trunk_imu: geometry 
- link trunk_imu_mount: geometry 
- link trunk_imu_sensing_point_x: geometry 
- link trunk_imu_sensing_point_y: geometry 
- link trunk_imu_sensing_point_z: geometry 

Commit message: [fix] Fix HyQReal model

File: resources/urdfs/hyqreal/urdf/hyqreal.urdf (robot description, URDF)
Before this commit: robot hyqreal, 43 links, 42 joints
Links:
- removed link base_link
- removed link realsense/back/camera_bottom_screw_frame
- removed link realsense/back/camera_color_frame
- removed link realsense/back/camera_color_optical_frame
- removed link realsense/back/camera_depth_frame
- removed link realsense/back/camera_depth_optical_frame
- removed link realsense/back/camera_left_ir_frame
- removed link realsense/back/camera_left_ir_optical_frame
- removed link realsense/back/camera_link
- removed link realsense/back/camera_right_ir_frame
- removed link realsense/back/camera_right_ir_optical_frame
- removed link realsense/front/camera_bottom_screw_frame
- removed link realsense/front/camera_color_frame
- removed link realsense/front/camera_color_optical_frame
- removed link realsense/front/camera_depth_frame
- removed link realsense/front/camera_depth_optical_frame
- removed link realsense/front/camera_left_ir_frame
- removed link realsense/front/camera_left_ir_optical_frame
- removed link realsense/front/camera_link
- removed link realsense/front/camera_right_ir_frame
- removed link realsense/front/camera_right_ir_optical_frame
- removed link trunk_imu
- removed link trunk_imu_mount
- removed link trunk_imu_sensing_point_x
- removed link trunk_imu_sensing_point_y
- removed link trunk_imu_sensing_point_z
Joints:
- removed joint floating_base
- removed joint realsense/back/camera_color_joint
- removed joint realsense/back/camera_color_optical_joint
- removed joint realsense/back/camera_depth_joint
- removed joint realsense/back/camera_depth_optical_joint
- removed joint realsense/back/camera_left_ir_joint
- removed joint realsense/back/camera_left_ir_optical_joint
- removed joint realsense/back/camera_link_joint
- removed joint realsense/back/camera_right_ir_joint
- removed joint realsense/back/camera_right_ir_optical_joint
- removed joint realsense/back/trunkcamera_joint
- removed joint realsense/front/camera_color_joint
- removed joint realsense/front/camera_color_optical_joint
- removed joint realsense/front/camera_depth_joint
- removed joint realsense/front/camera_depth_optical_joint
- removed joint realsense/front/camera_left_ir_joint
- removed joint realsense/front/camera_left_ir_optical_joint
- removed joint realsense/front/camera_link_joint
- removed joint realsense/front/camera_right_ir_joint
- removed joint realsense/front/camera_right_ir_optical_joint
- removed joint realsense/front/trunkcamera_joint
- removed joint trunk_imu_joint
- removed joint trunk_imu_mount_joint
- removed joint trunk_imu_sensing_point_x_joint
- removed joint trunk_imu_sensing_point_y_joint
- removed joint trunk_imu_sensing_point_z_joint
