Commit message: go1 resources

File: resources/urdfs/go1/urdf/go1.urdf (robot description, URDF)
Before this commit: robot go1, 36 links, 35 joints
Links:
- removed link world
- link trunk: geometry collision box size=0.52 0.22 0.14; visual mesh filename=package://go1_description/meshes/trunk.dae scale=1 1 1
Joints:
- removed joint floating_base_joint
- joint lf_haa_joint: limit lower=-6.283185307179586 upper=6.283185307179586 effort=2370 velocity=3000 -> lower=-0.863 upper=0.863 effort=23.7 velocity=30.1
- joint lf_hfe_joint: limit lower=-6.283185307179586 upper=6.283185307179586 effort=2370 velocity=3000 -> lower=-0.686 upper=4.501 effort=23.7 velocity=30.1
- joint lf_kfe_joint: limit lower=-6.283185307179586 upper=6.283185307179586 effort=2370 velocity=3000 -> lower=-2.818 upper=-0.888 effort=35.55 velocity=20.06
- joint lh_haa_joint: limit lower=-6.283185307179586 upper=6.283185307179586 effort=2370 velocity=3000 -> lower=-0.863 upper=0.863 effort=23.7 velocity=30.1
- joint lh_hfe_joint: limit lower=-6.283185307179586 upper=6.283185307179586 effort=2370 velocity=3000 -> lower=-0.686 upper=4.501 effort=23.7 velocity=30.1
- joint lh_kfe_joint: limit lower=-6.283185307179586 upper=6.283185307179586 effort=2370 velocity=3000 -> lower=-2.818 upper=-0.888 effort=35.55 velocity=20.06
- joint rf_haa_joint: limit lower=-6.283185307179586 upper=6.283185307179586 effort=2370 velocity=3000 -> lower=-0.863 upper=0.863 effort=23.7 velocity=30.1
- joint rf_hfe_joint: limit lower=-6.283185307179586 upper=6.283185307179586 effort=2370 velocity=3000 -> lower=-0.686 upper=4.501 effort=23.7 velocity=30.1
- joint rf_kfe_joint: limit lower=-6.283185307179586 upper=6.283185307179586 effort=2370 velocity=3000 -> lower=-2.818 upper=-0.888 effort=35.55 velocity=20.06
- joint rh_haa_joint: limit lower=-6.283185307179586 upper=6.283185307179586 effort=2370 velocity=3000 -> lower=-0.863 upper=0.863 effort=23.7 velocity=30.1
- joint rh_hfe_joint: limit lower=-6.283185307179586 upper=6.283185307179586 effort=2370 velocity=3000 -> lower=-0.686 upper=4.501 effort=23.7 velocity=30.1
- joint rh_kfe_joint: limit lower=-6.283185307179586 upper=6.283185307179586 effort=2370 velocity=3000 -> lower=-2.818 upper=-0.888 effort=35.55 velocity=20.06
